File: v1.0/Noduino-iBaihe.sch (EAGLE design)
At the start: 42 parts, among them IC1 5V, Q1 SI2302, Q2 SI2302, Q3 SI2302, Q4 SI2302, Q5 SI2302

Commit message: change the drill size of pins interface to 0.9mm
The old drill size of v1.0 shield is 0.7mm.
It's too small
Parts:
- N1: value NODUINO-PIN -> NODUINO-PINMAIL; device ehl:NODUINO-PIN -> ehl:NODUINO-PINMAIL
Changed lines of the file:
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@@
 <part name="PAD9" library="ehl" deviceset="2,15/1,0" device=""/>
 <part name="PAD10" library="ehl" deviceset="2,15/1,0" device=""/>
-<part name="N1" library="ehl" deviceset="NODUINO-PIN" device=""/>
+<part name="N1" library="ehl" deviceset="NODUINO-PIN" device="MAIL" value="NODUINO-PINMAIL"/>
 <part name="IC1" library="ehl" deviceset="AMS1117" device="SOT223" value="5V"/>
 <part name="GND12" library="ehl" deviceset="GND" device=""/>
